File: Prop_Fan.brd (EAGLE design)
At the start: 120 parts, among them J1 1546215-2, J2 1546215-2, J3 1546215-2, J4 1546215-2, SW2 EVQ-Q2203W, SW3 EVQ-Q2203W, SW4 EVQ-Q2203W, U1 P8X32A-Q44, U10 MAX31855KASA+, U11 MAX31855KASA+, U12 MF-DSC-SOT233-BSS138, U13 MF-DSC-SOT233-BSS138, U14 CD74HC595M96, U16 CD74HC165M96, U17 MF-DSC-SOT233-BSS138, U18 MF-DSC-SOT233-BSS138, U19 MF-DSC-SOT233-BSS138, U2 MF-DSC-SOT233-BSS138, U3 MF-DSC-SOT233-BSS138, U4 MAX31855KASA+, U5 LM22678TJ-5.0/NOPB, U6 ADP3338AKCZ-3.3-RL, U7 CAT24C512WI-GT3, U8 MF-DSC-SOT233-BSS138, U9 MAX31855KASA+, X1 ABMM-6.000MHZ-B2-T

Commit message: Working on Switch inputs. Voltage Dividers!
Parts:
- added R27, R31, R33, R35, R37, R39, R41, R43: 27K, MF_Passives:R0603
- added R28, R32, R34, R36, R38, R40, R42, R44: 10K, MF_Passives:R0603
Connections:
- net IN_OPTO_1: now also R27.P$1, R28.P$1
Changed lines of the file:
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@@
 <attribute name="LABEL01" value="RLY_0" x="-322" y="-506" size="1.778" layer="27" display="off"/>
+</element>
+<element name="R27" library="MF_Passives" package="R0603" value="27K" x="-334" y="-516.5">
+<attribute name="TOLERANCE" value="N/A" x="-334" y="-516.5" size="1.778" layer="27" display="off"/>
+<attribute name="MFG#" value="N/A" x="-334" y="-516.5" size="1.778" layer="27" display="off"/>
+<attribute name="VOLTAGE" value="N/A" x="-334" y="-516.5" size="1.778" layer="27" display="off"/>
+<attribute name="WATTAGE" value="N/A" x="-334" y="-516.5" size="1.778" layer="27" display="off"/>
+</element>
+<element name="R28" library="MF_Passives" package="R0603" value="10K" x="-334" y="-520">
+<attribute name="TOLERANCE" value="N/A" x="-334" y="-520" size="1.778" layer="27" display="off"/>
+<attribute name="MFG#" value="N/A" x="-334" y="-520" size="1.778" layer="27" display="off"/>
+<attribute name="VOLTAGE" value="N/A" x="-334" y="-520" size="1.778" layer="27" display="off"/>
+<attribute name="WATTAGE" value="N/A" x="-334" y="-520" size="1.778" layer="27" display="off"/>
+</element>
+<element name="R31" library="MF_Passives" package="R0603" value="27K" x="-334" y="-523.5">
+<attribute name="TOLERANCE" value="N/A" x="-334" y="-523.5" size="1.778" layer="27" display="off"/>
+<attribute name="MFG#" value="N/A" x="-334" y="-523.5" size="1.778" layer="27" display="off"/>
+<attribute name="VOLTAGE" value="N/A" x="-334" y="-523.5" size="1.778" layer="27" display="off"/>
+<attribute name="WATTAGE" value="N/A" x="-334" y="-523.5" size="1.778" layer="27" display="off"/>
+</element>
+<element name="R32" library="MF_Passives" package="R0603" value="10K" x="-334" y="-527">
+<attribute name="TOLERANCE" value="N/A" x="-334" y="-527" size="1.778" layer="27" display="off"/>
+<attribute name="MFG#" value="N/A" x="-334" y="-527" size="1.778" layer="27" display="off"/>
+<attribute name="VOLTAGE" value="N/A" x="-334" y="-527" size="1.778" layer="27" display="off"/>
+<attribute name="WATTAGE" value="N/A" x="-334" y="-527" size="1.778" layer="27" display="off"/>
+</element>
+<element name="R33" library="MF_Passives" package="R0603" value="27K" x="-334" y="-530.5">
+<attribute name="TOLERANCE" value="N/A" x="-334" y="-530.5" size="1.778" layer="27" display="off"/>
+<attribute name="MFG#" value="N/A" x="-334" y="-530.5" size="1.778" layer="27" display="off"/>
+<attribute name="VOLTAGE" value="N/A" x="-334" y="-530.5" size="1.778" layer="27" display="off"/>
+<attribute name="WATTAGE" value="N/A" x="-334" y="-530.5" size="1.778" layer="27" display="off"/>
+</element>
+<element name="R34" library="MF_Passives" package="R0603" value="10K" x="-334" y="-534">
+<attribute name="TOLERANCE" value="N/A" x="-334" y="-534" size="1.778" layer="27" display="off"/>
+<attribute name="MFG#" value="N/A" x="-334" y="-534" size="1.778" layer="27" display="off"/>
+<attribute name="VOLTAGE" value="N/A" x="-334" y="-534" size="1.778" layer="27" display="off"/>
+<attribute name="WATTAGE" value="N/A" x="-334" y="-534" size="1.778" layer="27" display="off"/>
+</element>
+<element name="R35" library="MF_Passives" package="R0603" value="27K" x="-334" y="-537.5">
+<attribute name="TOLERANCE" value="N/A" x="-334" y="-537.5" size="1.778" layer="27" display="off"/>
+<attribute name="MFG#" value="N/A" x="-334" y="-537.5" size="1.778" layer="27" display="off"/>
+<attribute name="VOLTAGE" value="N/A" x="-334" y="-537.5" size="1.778" layer="27" display="off"/>
+<attribute name="WATTAGE" value="N/A" x="-334" y="-537.5" size="1.778" layer="27" display="off"/>
+</element>
+<element name="R36" library="MF_Passives" package="R0603" value="10K" x="-334" y="-541">
+<attribute name="TOLERANCE" value="N/A" x="-334" y="-541" size="1.778" layer="27" display="off"/>
+<attribute name="MFG#" value="N/A" x="-334" y="-541" size="1.778" layer="27" display="off"/>
+<attribute name="VOLTAGE" value="N/A" x="-334" y="-541" size="1.778" layer="27" display="off"/>
+<attribute name="WATTAGE" value="N/A" x="-334" y="-541" size="1.778" layer="27" display="off"/>
+</element>
+<element name="R37" library="MF_Passives" package="R0603" value="27K" x="-334" y="-544.5">
+<attribute name="TOLERANCE" value="N/A" x="-334" y="-544.5" size="1.778" layer="27" display="off"/>
+<attribute name="MFG#" value="N/A" x="-334" y="-544.5" size="1.778" layer="27" display="off"/>
+<attribute name="VOLTAGE" value="N/A" x="-334" y="-544.5" size="1.778" layer="27" display="off"/>
+<attribute name="WATTAGE" value="N/A" x="-334" y="-544.5" size="1.778" layer="27" display="off"/>
+</element>
+<element name="R38" library="MF_Passives" package="R0603" value="10K" x="-330.5" y="-544.5">
+<attribute name="TOLERANCE" value="N/A" x="-334" y="-548" size="1.778" layer="27" display="off"/>
+<attribute name="MFG#" value="N/A" x="-334" y="-548" size="1.778" layer="27" display="off"/>
+<attribute name="VOLTAGE" value="N/A" x="-334" y="-548" size="1.778" layer="27" display="off"/>
+<attribute name="WATTAGE" value="N/A" x="-334" y="-548" size="1.778" layer="27" display="off"/>
+</element>
+<element name="R39" library="MF_Passives" package="R0603" value="27K" x="-334" y="-548">
+<attribute name="TOLERANCE" value="N/A" x="-334" y="-551.5" size="1.778" layer="27" display="off"/>
+<attribute name="MFG#" value="N/A" x="-334" y="-551.5" size="1.778" layer="27" display="off"/>
+<attribute name="VOLTAGE" value="N/A" x="-334" y="-551.5" size="1.778" layer="27" display="off"/>
+<attribute name="WATTAGE" value="N/A" x="-334" y="-551.5" size="1.778" layer="27" display="off"/>
+</element>
+<element name="R40" library="MF_Passives" package="R0603" value="10K" x="-330.5" y="-548">
+<attribute name="TOLERANCE" value="N/A" x="-334" y="-555" size="1.778" layer="27" display="off"/>
+<attribute name="MFG#" value="N/A" x="-334" y="-555" size="1.778" layer="27" display="off"/>
+<attribute name="VOLTAGE" value="N/A" x="-334" y="-555" size="1.778" layer="27" display="off"/>
+<attribute name="WATTAGE" value="N/A" x="-334" y="-555" size="1.778" layer="27" display="off"/>
+</element>
+<element name="R41" library="MF_Passives" package="R0603" value="27K" x="-334" y="-551.5">
+<attribute name="TOLERANCE" value="N/A" x="-334" y="-558.5" size="1.778" layer="27" display="off"/>
+<attribute name="MFG#" value="N/A" x="-334" y="-558.5" size="1.778" layer="27" display="off"/>
+<attribute name="VOLTAGE" value="N/A" x="-334" y="-558.5" size="1.778" layer="27" display="off"/>
+<attribute name="WATTAGE" value="N/A" x="-334" y="-558.5" size="1.778" layer="27" display="off"/>
+</element>
+<element name="R42" library="MF_Passives" package="R0603" value="10K" x="-330.5" y="-551.5">
+<attribute name="TOLERANCE" value="N/A" x="-334" y="-562" size="1.778" layer="27" display="off"/>
+<attribute name="MFG#" value="N/A" x="-334" y="-562" size="1.778" layer="27" display="off"/>
+<attribute name="VOLTAGE" value="N/A" x="-334" y="-562" size="1.778" layer="27" display="off"/>
+<attribute name="WATTAGE" value="N/A" x="-334" y="-562" size="1.778" layer="27" display="off"/>
+</element>
+<element name="R43" library="MF_Passives" package="R0603" value="27K" x="-334" y="-555">
+<attribute name="TOLERANCE" value="N/A" x="-334" y="-565.5" size="1.778" layer="27" display="off"/>
+<attribute name="MFG#" value="N/A" x="-334" y="-565.5" size="1.778" layer="27" display="off"/>
+<attribute name="VOLTAGE" value="N/A" x="-334" y="-565.5" size="1.778" layer="27" display="off"/>
+<attribute name="WATTAGE" value="N/A" x="-334" y="-565.5" size="1.778" layer="27" display="off"/>
+</element>
+<element name="R44" library="MF_Passives" package="R0603" value="10K" x="-330.5" y="-555">
+<attribute name="TOLERANCE" value="N/A" x="-334" y="-569" size="1.778" layer="27" display="off"/>
+<attribute name="MFG#" value="N/A" x="-334" y="-569" size="1.778" layer="27" display="off"/>
+<attribute name="VOLTAGE" value="N/A" x="-334" y="-569" size="1.778" layer="27" display="off"/>
+<attribute name="WATTAGE" value="N/A" x="-334" y="-569" size="1.778" layer="27" display="off"/>
 </element>
 </elements>
@@
 <signal name="IN_OPTO_1">
 <contactref element="U16" pad="12"/>
+<contactref element="R27" pad="P$1"/>
+<contactref element="R28" pad="P$1"/>
+<wire x1="-334.75" y1="-516.5" x2="-287.4" y2="-405.635" width="0" layer="19" extent="1-1"/>
+<wire x1="-334.75" y1="-520" x2="-334.75" y2="-516.5" width="0" layer="19" extent="1-1"/>
 </signal>
 <signal name="IN_OPTO_2">
