File: Hardware/Prop_Fan.sch (EAGLE design)
At the start: 136 parts, among them J1 1546215-2, J2 1546215-2, J3 1546215-2, J4 1546215-2, SW2 EVQ-Q2203W, SW3 EVQ-Q2203W, SW4 EVQ-Q2203W, U1 P8X32A-Q44, U10 MAX31855KASA+, U11 MAX31855KASA+, U12 MF-DSC-SOT233-BSS138, U13 MF-DSC-SOT233-BSS138, U14 CD74HC595M96, U16 CD74HC165M96, U17 MF-DSC-SOT233-BSS138, U18 MF-DSC-SOT233-BSS138, U19 MF-DSC-SOT233-BSS138, U2 MF-DSC-SOT233-BSS138, U3 MF-DSC-SOT233-BSS138, U4 MAX31855KASA+, U5 LM22678TJ-5.0/NOPB, U6 ADP3338AKCZ-3.3-RL, U7 CAT24C512WI-GT3, U8 MF-DSC-SOT233-BSS138, U9 MAX31855KASA+, X1 ABMM-6.000MHZ-B2-T

Commit message: IMU E-compass added. Routing almost done.
Need to add a way to look at the dome brightness.
Parts:
- removed D5, D6: MF-LED-0805-RED, PP_LED:LED_SINGLE_0805
- removed R43: 27K, MF_Passives:RESISTOR_0603
- removed R44, R47, R48, R49, R50, R51, R52: 10K, MF_Passives:RESISTOR_0603
- removed RELAYS1: 1-282834-0, PP_Connectors:CON_01X10_1-282834-0
- removed SW4: EVQ-Q2203W, PP_Electromechanical:SPST_EVQ-Q2203W
- added C13: C3225X7S2A475M200AB, PP_Passives:CAPACITOR_NON_POLAR_1210
- added C25, C26, C37, C40, C8: 0.1uF, PP_Passives:CAPACITOR_NON_POLAR_0805
- added C36: 4.7uF, PP_Passives:CAPACITOR_NON_POLAR_0805
- added SW1: MF-SW-TACT-4.2MM, MF_Switches:TACT_4.2MM
- added SWITCHS: 1-282834-0, PP_Connectors:CON_01X10_1-282834-0
- added SW_D, SW_S, SW_U: 1546215-2, PP_Connectors:CON_01X02_1546215-2
- added U15, U20, U21, U22, U23, U24, U25, U26: G3VM-61GR2(TR05), PP_DigitalIC:G3VM-61GR2
- added U27: FXOS8700CQR1, PP_Sensors:FXOS8700CQR1
- BOARD_PWR: value (none) -> 1546215-2; device PP_Connectors:CON_01X03_640454-3 -> PP_Connectors:CON_01X02_1546215-2; LABEL01 (none) -> 12V; LABEL02 (none) -> GND
- C17, C22, C6: device PP_Passives:CAPACITOR_NON_POLAR_0805 -> PP_Passives:CAPACITOR_NON_POLAR_1210
- C5: device PP_Passives:CAPACITOR_NON_POLAR_0805 -> PP_Passives:CAPACITOR_NON_POLAR_0603
- R11, R14, R18, R3, R4, R5, R6, R7, R8: device PP_Passives:RESISTOR_0805 -> PP_Passives:RESISTOR_0603
- R12: value 390 -> 10K; device PP_Passives:RESISTOR_0805 -> PP_Passives:RESISTOR_0603
- R13: value 1K -> 10K; device PP_Passives:RESISTOR_0805 -> PP_Passives:RESISTOR_0603
- R2: value 10K -> 470K; device PP_Passives:RESISTOR_0805 -> PP_Passives:RESISTOR_0603
- R27, R37, R39, R41: value 27K -> 1.2K
- R31, R33, R35: value 27K -> 10K
- R36, R38, R40, R42: value 10K -> 1.2K
- SW2, SW3: value EVQ-Q2203W -> MF-SW-TACT-4.2MM; device PP_Electromechanical:SPST_EVQ-Q2203W -> MF_Switches:TACT_4.2MM
- U12, U13, U17, U18, U19, U2, U3, U8: value MF-DSC-SOT233-BSS138 -> G3VM-61GR2(TR05); device MF_Discrete_Semiconductor:N-CHANNEL_FET_SOT-23-3 -> PP_DigitalIC:G3VM-61GR2
- renumbered D4 to 3.3V_PWR
Connections:
- net OUT_OPTO_0 renamed OUT_0
- net OUT_OPTO_1 renamed OUT_1
- net OUT_OPTO_2 renamed OUT_2
- net OUT_OPTO_3 renamed OUT_3
- net OUT_OPTO_4 renamed OUT_4
- net OUT_OPTO_5 renamed OUT_5
- net OUT_OPTO_6 renamed OUT_6
- net OUT_OPTO_7 renamed OUT_7
- removed net P$1: R29.P$1, R30.P$1, R47.P$1, R48.P$1, R49.P$1, R50.P$1, R51.P$1, R52.P$1, U12.SOURCE, U13.SOURCE, U17.SOURCE, U18.SOURCE, U19.SOURCE, U2.SOURCE, U3.SOURCE, U8.SOURCE
- removed net P19: U1.P19
- removed net P20: U1.P20
- removed net P21: U1.P21
- new net N$1: R28.P$1, U16.D0, U19.4
- new net N$10: R38.P$1, U22.ANODE
- new net N$19: R39.P$1, U23.ANODE
- new net N$20: R40.P$1, U24.ANODE
- new net N$21: R41.P$1, U25.ANODE
- new net N$22: R42.P$1, U26.ANODE
- new net N$23: R27.P$2, SWITCHS.1
- new net N$24: R36.P$2, SWITCHS.2
- new net N$25: R37.P$2, SWITCHS.3
- new net N$26: R38.P$2, SWITCHS.4
- new net N$27: R39.P$2, SWITCHS.5
- new net N$28: R40.P$2, SWITCHS.6
- new net N$29: R41.P$2, SWITCHS.7
- new net N$3: R27.P$1, U19.ANODE
- new net N$30: R42.P$2, SWITCHS.8
- new net N$31: R2.2, U5.EN
- new net N$4: R36.P$1, U20.ANODE
- new net N$6: R37.P$1, U21.ANODE
- new net P0: U1.P0
- new net SCL_1: R12.1, U1.P10, U27.SCL/SCKL
- new net SDA_1: R13.1, U1.P9, U27.SDA/MOSI
- new net T+_3: C12.1, D10.1, J4.PIN1, U4.T+
- new net T-_3: C12.2, D10.2, J4.PIN2, U4.T-
- net 12V_CLEAN: now also R2.1; no longer R13.2
- net 165_CLK: now also U1.P13; no longer U1.P14
- net 165_DATA: now also U1.P11; no longer U1.P15
- net 165_LOAD: now also U1.P12; no longer U1.P16
- net 3.3V: now also C25.1, C36.1, C37.1, C8.1, R12.2, R13.2, R28.P$2, R29.P$2, R30.P$2, R31.P$2, R32.P$2, R33.P$2, R34.P$2, R35.P$2, U27.VDD, U27.VDDIO; no longer R2.2
- net 595_CLK: now also U1.P16; no longer U1.P11
- net 595_DATA: now also U1.P14; no longer U1.P12
- net 595_LAT: now also U1.P15; no longer U1.P13
- net 5V_PWR: now also C13.1; no longer R12.2
- net CHASSIS_GND: now also BOARD_PWR.PIN2, U12.3, U13.3, U15.3, U17.3, U18.3, U19.CATHODE, U2.3, U20.CATHODE, U21.CATHODE, U22.CATHODE, U23.CATHODE, U24.CATHODE, U25.CATHODE, U26.CATHODE, U3.3, U8.3; no longer BOARD_PWR.PIN3
- net GND: now also C13.2, C25.2, C26.2, C36.2, C37.2, C40.2, C8.2, SW1.P$4, SW2.P$4, SW3.P$4, SW_D.PIN2, SW_S.PIN2, SW_U.PIN2, U12.CATHODE, U13.CATHODE, U15.CATHODE, U17.CATHODE, U18.CATHODE, U19.3, U2.CATHODE, U20.3, U21.3, U22.3, U23.3, U24.3, U25.3, U26.3, U27.GND, U27.RST, U27.SA0/MISO, U27.SA1/CS_B, U3.CATHODE, U8.CATHODE; no longer D5.CATHODE, D6.CATHODE, SW2.B, SW3.B, SW4.B
- net IN_OPTO_1: now also R29.P$1, U20.4; no longer R27.P$1, R28.P$1
- net IN_OPTO_2: now also R30.P$1, U21.4
- net IN_OPTO_3: now also R31.P$1, U22.4
- net IN_OPTO_4: now also R32.P$1, U23.4
- net IN_OPTO_5: now also R33.P$1, U24.4
- net IN_OPTO_6: now also R34.P$1, U25.4
- net IN_OPTO_7: now also R35.P$1, U26.4
- net N$11: now also U2.ANODE; no longer R29.P$2, U2.GATE
- net N$12: now also U3.ANODE; no longer R30.P$2, U3.GATE
- net N$13: now also U8.ANODE; no longer R47.P$2, U8.GATE
- net N$14: now also U12.ANODE; no longer R48.P$2, U12.GATE
- net N$15: now also U13.ANODE; no longer R49.P$2, U13.GATE
- net N$16: now also U15.ANODE; no longer R50.P$2, U17.GATE
- net N$17: now also U17.ANODE; no longer R51.P$2, U18.GATE
- net N$18: now also U18.ANODE; no longer R52.P$2, U19.GATE
- net N$7: now also C26.1, U27.BYP; no longer D6.ANODE, R13.1
- net N$8: now also C40.1, U27.CRST; no longer D5.ANODE, R12.1
- net PROP_D4: now also U1.P3; no longer U1.P7
- net PROP_D5: now also U1.P4; no longer U1.P8
- net PROP_D6: now also U1.P1; no longer U1.P9
- net PROP_D7: now also U1.P2; no longer U1.P10
- net PROP_E2: now also U1.P8; no longer U1.P6
- net PROP_R/W: now also U1.P6; no longer U1.P4
- net PROP_RES: no longer R2.1
- net PROP_RS: now also U1.P7; no longer U1.P3
- net RLY_0: now also U2.4; no longer U2.DRAIN
- net RLY_1: now also U3.4; no longer U3.DRAIN
- net RLY_2: now also U8.4; no longer U8.DRAIN
- net RLY_3: now also U12.4; no longer U12.DRAIN
- net RLY_4: now also U13.4; no longer U13.DRAIN
- net RLY_5: now also U15.4; no longer U17.DRAIN
- net RLY_6: now also U17.4; no longer U18.DRAIN
- net RLY_7: now also U18.4; no longer U19.DRAIN
- net SW_D: now also SW3.P$1, SW_D.PIN1, U1.P19; no longer SW4.A, U1.P2
- net SW_S: now also SW2.P$1, SW_S.PIN1, U1.P20; no longer SW3.A, U1.P1
- net SW_U: now also SW1.P$1, SW_U.PIN1, U1.P21; no longer SW2.A, U1.P0
- net T+_0: now also D8.1; no longer D8.2
- net T+_1: now also D9.1; no longer C39.1, D7.2, D9.2, J3.PIN1, U11.T+
- net T+_2: now also C39.1, D7.1, J3.PIN1, U11.T+; no longer C12.1, D10.2, J4.PIN1, U4.T+
- net T-_0: now also D8.2; no longer D8.1
- net T-_1: now also D9.2; no longer C39.2, D7.1, D9.1, J3.PIN2, U11.T-
- net T-_2: now also C39.2, D7.2, J3.PIN2, U11.T-; no longer C12.2, D10.1, J4.PIN2, U4.T-
- net TC_SCK: now also U1.P27; no longer U1.P26
- net TC_SO: now also U1.P26; no longer U1.P27
Other:
- moved on the sheet: C15, C16, C17, C22, C23, C24, C27, C7, C9, D3, R12, R13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

Commit message: PROP  Fan Rev 1 complete.
Parts:
- added C41, C42, C43: .1uF, PP_Passives:CAPACITOR_NON_POLAR_0603
- added C44, C45: 10uF, PP_Passives:CAPACITOR_NON_POLAR_1210
- added J5: 1546215-2, PP_Connectors:CON_01X02_1546215-2
- added R43, R44, R45: 220, MF_Passives:RESISTOR_0603
- added U28: ACPL-C870-000E, PP_AnalogIC:ACPL-C87X
- added U29: MAX11613EUA+, PP_AnalogIC:MAX11613EUA+
- added U30: TPS7B6950QDBVRQ1, MF_IC_Power:TPS7B69
Connections:
- new net A0: R43.P$2, U29.A_0
- new net A1: U29.A_1
- new net A2: U29.A_2
- new net A3: U29.A_3
- new net EXT_5V: C45.1, U28.VDD1, U30.VOUT
- new net N$32: C42.1, R43.P$1, U28.VOUT+
- new net N$33: R44.P$2, R45.P$2, U28.VIN
- new net N$36: J5.PIN1, R45.P$1
- net 12V_BATT_ON: now also C44.1, U30.VIN
- net 3.3V: now also C41.1, C43.1, U28.VDD2, U29.VCC
- net CHASSIS_GND: now also C44.2, C45.2, R44.P$1, U28.GND1, U28.SHDN, U30.GND/ADJ
- net GND: now also C41.2, C42.2, C43.2, U28.GND2, U28.VOUT-, U29.GND
- net SCL_1: now also U29.SCL
- net SDA_1: now also U29.SDA

Commit message: Fixed a couple traces and added camfiles.
Parts:
- added U$35: JEEP_LOGO_SILK_MEDIUM, PP_Aesthetics:JEEP_LOGO_SILK_MEDIUM
- added U$42: LHE_LOGOLHE_LOGO, PP_Aesthetics:LHE_LOGOLHE_LOGO
Changed lines of the file:
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@@
 <?xml version="1.0" encoding="utf-8"?>
 <!DOCTYPE eagle SYSTEM "eagle.dtd">
-<eagle version="7.4.0">
+<eagle version="6.6.0">
 <drawing>
 <settings>
@@
 <part name="C45" library="PP_Passives" deviceset="CAPACITOR_NON_POLAR" device="_1210" value="10uF"/>
 <part name="U30" library="MF_IC_Power" deviceset="TPS7B69" device="" value="TPS7B6950QDBVRQ1"/>
+<part name="U$35" library="PP_Aesthetics" deviceset="JEEP_LOGO" device="_SILK_MEDIUM"/>
+<part name="U$42" library="PP_Aesthetics" deviceset="LHE_LOGO" device="LHE_LOGO"/>
 </parts>
 <sheets>
@@
 <instance part="C45" gate="G$1" x="472.44" y="12.7"/>
 <instance part="U30" gate="G$1" x="457.2" y="20.32"/>
+<instance part="U$35" gate="G$1" x="213.36" y="-45.72"/>
+<instance part="U$42" gate="G$1" x="213.36" y="-43.18" rot="MR0"/>
 </instances>
 <busses>

Commit message: Fixed VFD connector. Was mirrored.
Changed lines of the file:
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@@
 <?xml version="1.0" encoding="utf-8"?>
 <!DOCTYPE eagle SYSTEM "eagle.dtd">
-<eagle version="6.6.0">
+<eagle version="7.4.0">
 <drawing>
 <settings>
