File: Hardware/Cyclone-Pulse-Wrangler-Mainboard.sch (EAGLE design)
At the start: 69 parts, among them J1 DF11G-16DP-2V(50), J2 TBL009-254-02GY-2GY, U1 P8X32A-Q44, U2 CAT24C512WI-GT3, U3 LT8672EMS#PBF, U4 LT8614IUDC#PBF, U5 LT8614IUDC#PBF, U6 IPD100N06S403ATMA2, U7 LTC2986HLX-1#PBF, U8 TXB0104DR, X1 6.0MHz

Commit message: updating board files
Parts:
- removed C22, C32: 10nF, PP_Passives:CAPACITOR_NON_POLAR_0603
- removed C23, C33: 47uF, PP_Passives:CAPACITOR_NON_POLAR_1210
- removed C24, C27, C30: 1uF, PP_Passives:CAPACITOR_NON_POLAR_0805
- removed C25, C26, C34: 10uF, PP_Passives:CAPACITOR_NON_POLAR_1210
- removed C28: 4.7pF, PP_Passives:CAPACITOR_NON_POLAR_0603
- removed C29: 0.1uF, PP_Passives:CAPACITOR_NON_POLAR_0603
- removed C31, C35, C36: 0.1uF, PP_Passives:CAPACITOR_NON_POLAR_0805
- removed FTDI_CABLE: (no value), PP_Connectors:CON_01X06_2.54MM_PIN_HEADER
- removed R11, R30: 1M, PP_Passives:RESISTOR_0603
- removed R28: 412K, PP_Passives:RESISTOR_0603
- removed R29: 41.2K, PP_Passives:RESISTOR_0603
- removed R31: 243K, PP_Passives:RESISTOR_0603
- removed TAG_CONNECT: TC2030-NL, PP_Connectors:CON_02X03_TC2030
- removed U8: TXB0104DR, PP_DigitalIC:TXB0104DR
- added D2: TPSMB33A, PP_Passives:DIODE_DO-214AA
- added D4: TPSMB18A, PP_Passives:DIODE_DO-214AA
- added D5: BZT52C3V6-TP, PP_Passives:DIODE_SOD-123
- added F1, F2, F3: (no value), PP_Passives:PTC_FUSE_2920
- added J3: MF-CON-2.54mm-01x01, MF_Connectors:CON_01X01_PTH_2.54MM
- added J4: RJHSE-538X, PP_Connectors:RJ45_SINGLE_RJHSE-538X
- added JMP1: 0, MF_Passives:RESISTOR_0603
- added LUG1, LUG2: B4A-PCB-RLM-KIT, PP_Connectors:CON_01X01_B4A-PCB-RLM
- added R6, R7: 5.1K, MF_Passives:RESISTOR_0603
- added SW1: MF-SW-TACT-4.2MM, MF_Switches:TACT_4.2MM
- added TC1: TC2030-IDC-NL, MF_Connectors:CON_02X03_SWD2TC_TC2030-IDC-NL
- C1, C18, C4, C6: value 0.1uF -> 1uF; MPN MF-CAP-0805-0.1uF -> C0805X105K5RACAUTO
- C11, C12, C19, C7: MPN MF-CAP-0805-0.1uF -> (none)
- C14: value 1uF -> 0.1uF; MPN C0805X105K5RACAUTO -> (none)
- C15: value 1uF -> 10uF; device PP_Passives:CAPACITOR_NON_POLAR_0805 -> PP_Passives:CAPACITOR_NON_POLAR_1210; MPN C0805X105K5RACAUTO -> (none)
- C16: value 4.7pF -> 0.1uF; device PP_Passives:CAPACITOR_NON_POLAR_0603 -> PP_Passives:CAPACITOR_NON_POLAR_0805; MPN C0603C479D5HACTU -> (none)
- C17: device PP_Passives:CAPACITOR_NON_POLAR_0603 -> PP_Passives:CAPACITOR_NON_POLAR_0805; MPN MF-CAP-0603-0.1uF -> (none)
- C2, C3: value 0.1uF -> 12pF; MPN MF-CAP-0805-0.1uF -> C0805X105K5RACAUTO
- C20: value 1uF -> 0.1uF; MPN MF-CAP-0805-1uF -> (none)
- C5: device PP_Passives:CAPACITOR_NON_POLAR_0603 -> PP_Passives:CAPACITOR_NON_POLAR_0805; MPN MF-CAP-0805-0.1uF -> (none)
- C8: value 0.1uF -> 10uF; device PP_Passives:CAPACITOR_NON_POLAR_0805 -> PP_Passives:CAPACITOR_NON_POLAR_1210; MPN MF-CAP-0805-0.1uF -> (none)
- J1: value DF11G-16DP-2V(50) -> TYPE-C-31-M-12; device PP_Connectors:CON_02X08_DF11G-16DP-2V(50) -> PP_Connectors:USB_TYPE-C_MINIMAL; LABEL01 LCD RX -> (none); LABEL02 LCD TX -> (none); LABEL15 GND -> (none); LABEL16 5V -> (none); MPN DF11G-16DP-2V(50) -> TYPE-C-31-M-12
- J2: value TBL009-254-02GY-2GY -> MF-CON-2.54mm-01x02; device PP_Connectors:CON_01X02_TBL009-254-02GY-2GY -> MF_Connectors:CON_01X02_PTH_2.54MM; LABEL01 +12V -> (none); LABEL02 GND -> (none)
- L2, L3: value IHLP2525CZER4R7M01 -> MI0603K300R-10; device PP_Passives:INDUCTOR_IHLP-2525 -> MF_Passives:INDUCTOR_0603; MPN IHLP2525CZER4R7M01 -> MI0603K300R-10
- R1: device PP_Passives:RESISTOR_0805 -> MF_Passives:RESISTOR_0603; MPN (none) -> MF-RES-0603-10K
- R2: value 41.2K -> 5.1K; device PP_Passives:RESISTOR_0603 -> MF_Passives:RESISTOR_0603
- R3: value 10K -> 100; device PP_Passives:RESISTOR_0603 -> MF_Passives:RESISTOR_0603; MPN MF-RES-0603-10K -> MF-RES-0603-100
- R4: value 10K -> 5.1K; device PP_Passives:RESISTOR_0603 -> MF_Passives:RESISTOR_0603; MPN MF-RES-0603-10K -> (none)
- R5: value 18K -> 10K; device PP_Passives:RESISTOR_0603 -> MF_Passives:RESISTOR_0603; MPN (none) -> MF-RES-0603-10K
- U1: value P8X32A-Q44 -> ATSAMD21G18A; device MF_IC_Digital:P8X32A-Q44 -> PP_DigitalIC:ATSAMD21G18A-AU; MPN (none) -> ATSAMD21G18A-AU; POPULATE (none) -> 1
- U2: value CAT24C512WI-GT3 -> IP4234CZ6,125; device PP_DigitalIC:EEPROM_I2CSOIC-8_W -> PP_Passives:IP4234CZ6; MPN CAT24C512WI-GT3 -> IP4234CZ6,125; POPULATE (none) -> 1; SPICEPREFIX X -> (none)
- U4: value LT8614IUDC#PBF -> NCP1117DT33G; device PP_PowerIC:LT8614IUDC#PBF -> PP_PowerIC:LINEAR_VOTLAGE_REGULATORS_NCP1117DT; MPN LT8614IUDC#PBF -> (none)
- U5: value LT8614IUDC#PBF -> ACS72981LLRATR-100U3; device PP_PowerIC:LT8614IUDC#PBF -> PP_Sensors:ACS72981; MPN LT8614IUDC#PBF -> ACS72981LLRATR-100U3
- U7: value LTC2986HLX-1#PBF -> PCA9615DP; device PP_Sensors:LTC2986HLX#PBF -> PP_DigitalIC:PCA9615DP; MPN LTC2986HLX-1#PBF -> (none)
- X1: value 6.0MHz -> ABS25-32.768KHZ-T; device MF_Frequency_Control:CYRSTAL_GND_ABMM -> MF_Frequency_Control:CYRSTAL_ABS25; MPN ABMM-6.000MHZ-B2-T -> ABS25-32.768KHZ-T
Connections:
- removed net !RES!_PROP: C5.1, FTDI_CABLE.6, TAG_CONNECT.PIN6
- removed net 3.3V_!CS: U1.P7, U8.A1
- removed net 3.3V_SCK: U1.P10, U8.A4
- removed net 3.3V_SDI: U1.P8, U8.A2
- removed net 3.3V_SDO: U1.P9, U8.A3
- removed net 5.0V: C11.1, C12.1, C18.1, C28.1, C33.1, C35.1, C6.1, C7.1, J1.16, L3.P$2, R30.2, U5.BIAS, U7.!RESET, U7.VDD, U8.VCCB
- removed net 5V_!CS: U7.!CS, U8.B1
- removed net 5V_SCK: U7.SCK, U8.B4
- removed net 5V_SDI: U7.SDI, U8.B2
- removed net 5V_SDO: U7.SDO, U8.B3
- removed net BST: C17.1, U4.BST
- removed net BST1: C29.1, U5.BST
- removed net FB: C16.2, R11.1, R28.2, U4.FB
- removed net FB1: C28.2, R30.1, R31.2, U5.FB
- removed net GPIO0: J1.11
- removed net GPIO1: J1.12
- removed net GPIO2: J1.9
- removed net GPIO3: J1.10
- removed net GPIO4: J1.13
- removed net INTVCC: C21.2, U4.INTVCC
- removed net INTVCC1: C30.2, U5.INTVCC
- removed net LCD_RX: J1.1, U1.P1
- removed net LCD_TX: J1.2, U1.P0
- removed net LTC2986_INTERRUPT: R4.1, R5.2, U1.P12
- removed net N$12: R4.2, U7.INTERRUPT
- removed net N$13: C10.1, C13.POS, C14.1, C15.1, C24.1, C27.1, C9.1, L1.P$1, U3.DRAIN, U4.EN/UV, U4.VIN1, U4.VIN2, U5.EN/UV, U5.VIN1, U5.VIN2, U6.DRAIN
- removed net N$6: C25.2, U7.Q2
- removed net N$7: C25.1, U7.Q1
- removed net N$8: C34.1, U7.LDO
- removed net P13: U1.P13
- removed net P14: U1.P14
- removed net P15: U1.P15
- removed net P16: U1.P16
- removed net P17: U1.P17
- removed net P18: U1.P18
- removed net P19: U1.P19
- removed net P2: U1.P2
- removed net P20: U1.P20
- removed net P21: U1.P21
- removed net P22: U1.P22
- removed net P23: U1.P23
- removed net P24: U1.P24
- removed net P25: U1.P25
- removed net P26: U1.P26
- removed net P27: U1.P27
- removed net P3: U1.P3
- removed net P4: U1.P4
- removed net P5: U1.P5
- removed net P6: U1.P6
- removed net PROP_RES: C5.2, R1.1, U1.RES'
- removed net RT: R2.2, U4.RT
- removed net RT1: R29.2, U5.RT
- removed net RX_PROP: FTDI_CABLE.4, TAG_CONNECT.PIN4, U1.P31
- removed net SCL: U1.P28, U2.SCL
- removed net SDA: U1.P29, U2.SDA
- removed net SPI_LEVEL_SHIFTER_OE: R3.2, U1.P11, U8.OE
- removed net SW: C17.2, L2.P$1, U4.SW
- removed net SW1: C29.2, L3.P$1, U5.SW
- removed net TR/SS: C22.2, U4.TR/SS
- removed net TR/SS1: C32.2, U5.TR/SS
- removed net TX_PROP: FTDI_CABLE.5, TAG_CONNECT.PIN3, U1.P30
- removed net VIN: D1.CATHODE, J2.PIN1, U3.SOURCE, U6.SOURCE
- removed net X0: U1.X0, X1.X1
- removed net X1: U1.X1, X1.X0
- new net !RESET: R1.P$2, R3.P$1, SW1.P$1, TC1.PIN6
- new net 12V: C10.1, C13.POS, C9.1, J2.PIN2, JMP1.P$1, L1.P$1, U3.DRAIN, U6.DRAIN
- new net 12V_FAN+: LUG2.PIN1, U5.IP-
- new net 12V_PWR: D1.CATHODE, F1.P$1, LUG1.PIN1, U5.IP+
- new net 12V_SW: D2.CATHODE, F2.P$1
- new net 3.3V_SCREEN_OUT: C21.1, D5.CATHODE, F3.P$1, J4.6
- new net A1: U1.PB8/EIC/AIN2/SCOM4PAD0/TC4
- new net A2: U1.PB9/EIC/AIN3/SCOM4PAD1/TC4
- new net A3: U1.PA4/EIC/REF/AIN4/SCOM0PAD0/TC0
- new net A4: U1.PA5/EIC/AIN5/SCOM0PAD1/TC0
- new net A5: U1.PB2/EIC/AIN10/SCOM5PAD0
- new net AREF: C6.1, U1.PA3/EIC/REF/AIN1
- new net CC1: J1.CC1, R2.P$1
- new net CC2: J1.CC2, R4.P$1
- new net D+: J1.D+, U2.I/O2B
- new net D-: J1.D-, U2.I/O1B
- new net D0: U1.PA11/EIC/AIN19/SCOM2PAD3/TC1
- new net D1: U1.PA10/EIC/AIN18/SCOM2PAD2/TC1
- new net D10: U1.PA18/EIC/SCOM1PAD2/TC3
- new net D11: U1.PA16/I2C/EIC/SCOM1PAD0/TC1
- new net D12: U1.PA19/EIC/SCOM1PAD3/TC3
- new net D13: U1.PA17/I2C/EIC/SCOM1PAD1/TC2
- new net D18: U1.PA22/I2C/EIC/SCOM5PAD0/TC4
- new net D19: U1.PA23/I2C/EIC/SCOM5PAD1/TC4
- new net D2: U1.PA14/XIN/EIC/SCOM2PAD2/TC3
- new net D3: U1.PA9/I2C/EIC/AIN17/SCOM2PAD1/TC0
- new net D4: U1.PA8/I2C/AIN16/SCOM2PAD0/TC0
- new net D5: U1.PA15/XOUT/EIC/SCOM2PAD3/TC3
- new net D6: U1.PA20/EIC/SCOM5PAD2
- new net D7: U1.PA21/EIC/SCOM5PAD3
- new net D8: U1.PA6/EIC/AIN6/SCOM0PAD2/TC1
- new net D9: U1.PA7/EIC/AIN7/SCOM0PAD3/TC1
- new net DM: U1.PA24/EIC/SCOM3PAD2/TC5, U2.I/O1A
- new net DP: U1.PA25/EIC/SCOM3PAD3/TC5, U2.I/O2A
- new net DSCLM: J4.4, U7.DSCLM
- new net DSCLP: J4.3, U7.DSCLP
- new net DSDAM: J4.2, U7.DSDAM
- new net DSDAP: J4.1, U7.DSDAP
- new net FAN_CURRENT: C17.1, U1.PA2/EIC/AIN0, U5.VIOUT
- new net PA12: U1.PA12/I2C/EIC/SCOM2PAD0/TC2
- new net PA13: U1.PA13/I2C/EIC/SCOM2PAD1/TC2
- new net PA27: U1.PA27/EIC
- new net PA28: U1.PA28/EIC
- new net PB22: U1.PB22/EIC/SCOM5PAD2
- new net PB23: U1.PB23/EIC/SCOM5PAD3
- new net PB3: U1.PB3/EIC/AIN11/SCOM5PAD1
- new net REG_INPUT: C8.1, J2.PIN1, JMP1.P$2, U4.IN
- new net RESETLIN: R3.P$2, U1.!RESET
- new net SCL_SCREEN: R6.P$1, U1.PB11/EIC/SCOM4PAD3/TC5, U7.SCL
- new net SDA_SCREEN: R7.P$1, U1.PB10/EIC/SCOM4PAD2/TC5, U7.SDA
- new net SHLD: J1.SHLD, L3.P$1
- new net SWCLK: TC1.PIN4, U1.PA30/EIC/SCOM1PAD2/TC1
- new net SWDIO: TC1.PIN3, U1.PA31/EIC/SCOM1PAD3/TC1
- new net SWO: TC1.PIN5
- new net USB_VBUS: C4.1, C5.1, J3.PIN1, L2.P$2, U2.VB
- new net USB_VBUS_PORT: J1.VBUS, L2.P$1
- new net VDDCORE: C1.1, U1.VDDCORE1
- new net XIN32: C2.2, U1.PA0/XIN32/EIC/SCOM1PAD0/TC2, X1.X0
- new net XOUT32: C3.2, U1.PA1/XOUT32/EIC/SCOM1PAD1/TC2, X1.X1
- net 3.3V: now also C11.1, C12.1, C14.1, C15.1, C18.1, C19.1, C20.1, C7.1, F3.P$2, R1.P$1, R6.P$2, R7.P$2, TC1.PIN1, U1.VDDANA, U1.VDDIN, U1.VDDIO1, U1.VDDIO2, U4.OUT, U5.VCC, U7.EN, U7.VDD; no longer C1.1, C2.1, C23.1, C3.1, C31.1, C36.1, C4.1, C8.1, L2.P$2, R1.2, R11.2, U1.VDD, U2.VCC, U4.BIAS, U8.VCCA
- net GND: now also C16.2, C17.2, C2.1, C21.2, C3.1, C5.2, D4.CATHODE, D5.ANODE, J1.GND, J4.5, L3.P$2, R2.P$2, R4.P$2, R5.P$1, SW1.P$3, TC1.PIN2, U1.GND, U7.VSS; no longer C2.2, C21.1, C22.1, C23.2, C24.2, C26.2, C27.2, C3.2, C30.1, C31.2, C32.1, C33.2, C34.2, C35.2, C36.2, FTDI_CABLE.1, J1.15, J2.PIN2, R2.1, R28.1, R29.1, R3.1, R31.1, R5.1, TAG_CONNECT.PIN5, U1.BOE', U1.VSS, U2.A1, U2.A2, U2.WP, U4.GND1, U4.GND2, U5.GND1, U5.GND2, U7.GND, U8.GND, X1.GND
- net N$1: now also D2.ANODE, D4.ANODE; no longer C19.1, U7.VREF_BYP
- net N$3: now also F1.P$2, U3.SOURCE, U6.SOURCE; no longer C20.1, U7.VREFOUT, U7.VREFP
- net N$4: now also F2.P$2, R5.P$2, U3.EN/UVLO; no longer C26.1, U7.Q3
Other:
- moved on the sheet: C1, C10, C11, C12, C13, C14, C15, C16, C17, C18, C19, C2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
