File: Hardware/Engine/Engine_Board.brd (EAGLE design)
At the start: 152.9 x 71.1 mm, 163 parts, among them J1 1546215-2, J2 1546215-2, J3 1546215-2, J4 1546215-2, J5 1546215-2, SW1 MF-SW-TACT-4.2MM, SW2 MF-SW-TACT-4.2MM, SW3 MF-SW-TACT-4.2MM, U1 P8X32A-Q44, U10 MAX31855KASA+, U11 MAX31855KASA+, U12 G3VM-61GR2(TR05), U13 G3VM-61GR2(TR05), U14 CD74HC595M96, U15 G3VM-61GR2(TR05), U16 CD74HC165M96, U17 G3VM-61GR2(TR05), U18 G3VM-61GR2(TR05), U19 G3VM-61GR2(TR05), U2 G3VM-61GR2(TR05), U20 G3VM-61GR2(TR05), U21 G3VM-61GR2(TR05), U22 G3VM-61GR2(TR05), U23 G3VM-61GR2(TR05), U24 G3VM-61GR2(TR05), U25 G3VM-61GR2(TR05), U26 G3VM-61GR2(TR05), U27 FXOS8700CQR1, U28 ACPL-C870-000E, U29 MAX11613EUA+, U3 G3VM-61GR2(TR05), U30 TPS7B6950QDBVRQ1, U4 MAX31855KASA+, U5 LM22678TJ-5.0/NOPB, U6 ADP3338AKCZ-3.3-RL, U7 CAT24C512WI-GT3, U8 G3VM-61GR2(TR05), U9 MAX31855KASA+, X1 ABMM-6.000MHZ-B2-T

Commit message: Working on new version
Parts:
- removed BOARD_PWR: 1546215-2, PP_Connectors:1546215-2
- removed C20: UWZ1H221MCL1GS, PP_Passives:10MM_CAP_SMD
- removed C21: UBW1H102MHD, PP_Passives:12.5MM_CAP_PTH
- removed L2: PLT10HH401100PNL, PP_Passives:PLT10H
- removed TP3, TP5: 5115-5119, PP_Connectors:KEYSTONE_5115-5119
- added J6: 3PCV-03-006, PP_Connectors:3PCV-03-006
- 12V, 3.3V, 5V, GND: value 5115-5119 -> (none)
- C10, C13, C29, C30: value C3225X7S2A475M200AB -> 4.7uF
- C14: value GRM21BR71H105KA12L -> 1uf
- C15: value UWZ1A102MCL1GS -> 1000uF
- C17: device PP_Passives:1210 -> PP_Passives:1206
- C18: value UBW1H102MHD -> 1000uF
- C19: value UWZ1H221MCL1GS -> 220uF
- C24: value UWJ1C470MCL1GB -> 47uF
- C27: value C0805C103K5RACTU -> 0.01uF
- C28: value 16SVP180M -> 180uF
- D2: value VS-12CWQ10FNPBF -> VS-12CWQ10FN-M3
- FID1, FID2: value FIDUCIAL_0.5MM -> (none)
- J1, J2, J3, J4, J5, SW_D, SW_S, SW_U: value 1546215-2 -> (none)
- L3: value IHLP5050CEER6R8M01 -> 6.8uH
- PROP_TC: value TC2030-FTDI-TTL-232R -> TC2030-NL
- R19, R20, R21, R22, R23, R24, R25, R26, R43, R44, R45: value 220 -> (none)
- R27, R36, R37, R38, R39, R40, R41, R42: value 1.2K -> (none)
- R28, R29, R30, R31, R32, R33, R34, R35: value 10K -> (none)
- RELAYS, SWITCHS: value 1-282834-0 -> (none)
- U30: value TPS7B6950QDBVRQ1 -> TPS7B6933QDCYRQ1
- renumbered TP1 to 5V, TP2 to 3.3V, TP4 to 12V, TP6 to GND
Connections:
- removed net 12V_CLEAN: C10.1, C14.1, C20.POS, C21.POS, C29.1, C30.1, L2.2, R2.1, TP3.P$1, U5.P$2
- new net 12V: 12V.P$1, C10.1, C14.1, C18.POS, C19.POS, C29.1, C30.1, D2.PAD-4, R2.1, U5.P$2
- new net 5V: 5V.P$1, C13.1, C15.POS, C16.1, C17.1, C28.POS, L3.1, U5.P$6, U6.3
- new net DOME_PWR: J6.3
- net 12V_BATT: now also J6.1; no longer BOARD_PWR.P$1
- net 12V_BATT_ON: no longer 12V.P$1, C18.POS, C19.POS, D2.PAD-4, L2.1
- net 3.3V: now also R11.1; no longer R11.2
- net 5V_PWR: no longer 5V.P$1, C13.1, C15.POS, C16.1, C17.1, C28.POS, L3.1, U5.P$6, U6.3
- net CHASSIS_GND: no longer BOARD_PWR.P$2, C18.NEG, C19.NEG, GND.P$1, L2.4, TVS1.P$1
- net GND: now also C18.NEG, C19.NEG, GND.P$1, J6.2, TVS1.P$1; no longer C20.NEG, C21.NEG, L2.3, TP5.P$1
- net N$9: now also R11.2; no longer R11.1
Routing:
- net 5V: track 0.00 -> 9.37 mm
- net 5V_PWR: track 28.4 -> 19.0 mm
- net 12V_BATT_ON: track 55.7 -> 52.7 mm
- net 12V_CLEAN: track 2.60 -> 0.00 mm
- net 12V: track 0.00 -> 2.60 mm
- net 3.3V: track 313.5 -> 311.6 mm
- net N$9: track 1.91 -> 0.00 mm
- net GND: track 189.0 -> 187.2 mm, vias 139 -> 138
- net N$5: track 2.96 -> 2.29 mm
- added copper zone on layer 1, net 12V
- removed copper zone on layer 1, net 12V_CLEAN
