File: Hardware/Engine/Engine_Board.sch (EAGLE design)
At the start: 159 parts, among them J1 1546215-2, J2 1546215-2, J3 1546215-2, J4 1546215-2, J5 1546215-2, SW1 MF-SW-TACT-4.2MM, SW2 MF-SW-TACT-4.2MM, SW3 MF-SW-TACT-4.2MM, U1 P8X32A-Q44, U10 MAX31855KASA+, U11 MAX31855KASA+, U12 G3VM-61GR2(TR05), U13 G3VM-61GR2(TR05), U14 CD74HC595M96, U15 G3VM-61GR2(TR05), U16 CD74HC165M96, U17 G3VM-61GR2(TR05), U18 G3VM-61GR2(TR05), U19 G3VM-61GR2(TR05), U2 G3VM-61GR2(TR05), U20 G3VM-61GR2(TR05), U21 G3VM-61GR2(TR05), U22 G3VM-61GR2(TR05), U23 G3VM-61GR2(TR05), U24 G3VM-61GR2(TR05), U25 G3VM-61GR2(TR05), U26 G3VM-61GR2(TR05), U27 FXOS8700CQR1, U28 ACPL-C870-000E, U29 MAX11613EUA+, U3 G3VM-61GR2(TR05), U30 TPS7B6950QDBVRQ1, U4 MAX31855KASA+, U5 LM22678TJ-5.0/NOPB, U6 ADP3338AKCZ-3.3-RL, U7 CAT24C512WI-GT3, U8 G3VM-61GR2(TR05), U9 MAX31855KASA+, X1 ABMM-6.000MHZ-B2-T

Commit message: Working on new version
Parts:
- removed BOARD_PWR: 1546215-2, PP_Connectors:CON_01X02_1546215-2
- removed C20: UWZ1H221MCL1GS, PP_Passives:CAPACITOR_POLARIZED_10MM_SMD
- removed C21: UBW1H102MHD, PP_Passives:CAPACITOR_POLARIZED_12.5MM_PTH
- removed L2: PLT10HH401100PNL, PP_Passives:COMMON_MODE_INDUCTOR_PLT10H
- removed TP1, TP2, TP3, TP4, TP5, TP6: 5115-5119, PP_Connectors:TEST_POINT_SINGLE_KEYSTONE_5115-5119
- added 12V, 3.3V, 5V, GND: (no value), PP_Connectors:TEST_POINT_SINGLE_KEYSTONE_5115-5119
- added J6: 3PCV-03-006, PP_Connectors:CON_01X03_3PV-03-006
- 3.3V_PWR: MPN (none) -> MF-LED-0805-RED
- C10, C13, C29, C30: value C3225X7S2A475M200AB -> 4.7uF; MPN (none) -> GRJ32DC72A475KE11L
- C14: value GRM21BR71H105KA12L -> 1uf; MPN (none) -> C0805C105K5RACTU
- C15: value UWZ1A102MCL1GS -> 1000uF; MPN (none) -> UWZ1A102MCL1GS
- C16, C23: MPN (none) -> MF-CAP-0805-0.1uF
- C17: device PP_Passives:CAPACITOR_NON_POLAR_1210 -> PP_Passives:CAPACITOR_NON_POLAR_1206; MPN (none) -> MF-CAP-1206-10uF
- C18: value UBW1H102MHD -> 1000uF; MPN (none) -> UBW1H102MHD
- C19: value UWZ1H221MCL1GS -> 220uF; MPN (none) -> UWZ1H221MCL1GS
- C22: MPN (none) -> MF-CAP-1206-10uF
- C24: value UWJ1C470MCL1GB -> 47uF; MPN (none) -> UWJ1C470MCL1GB
- C27: value C0805C103K5RACTU -> 0.01uF; MPN (none) -> C0805C103K5RACTU
- C28: value 16SVP180M -> 180uF; MPN (none) -> 16SVP180M
- D2: value VS-12CWQ10FNPBF -> VS-12CWQ10FN-M3; MPN (none) -> VS-12CWQ10FN-M3
- J1, J2, J3, J4, J5, SW_D, SW_S, SW_U: value 1546215-2 -> (none)
- L3: value IHLP5050CEER6R8M01 -> 6.8uH; MPN (none) -> IHLP5050CEER6R8M01
- PROP_TC: value TC2030-FTDI-TTL-232R -> TC2030-NL
- R11: MPN (none) -> MF-RES-0603-330
- R19, R20, R21, R22, R23, R24, R25, R26, R43, R44, R45: value 220 -> (none)
- R2: MPN (none) -> MF-RES-0603-470K
- R27, R36, R37, R38, R39, R40, R41, R42: value 1.2K -> (none)
- R28, R29, R30, R31, R32, R33, R34, R35: value 10K -> (none)
- RELAYS, SWITCHS: value 1-282834-0 -> (none)
- U30: value TPS7B6950QDBVRQ1 -> TPS7B6933QDCYRQ1; device MF_IC_Power:TPS7B69 -> MF_IC_Power:TPS7B6933QDCYRQ1
- U5: MPN (none) -> LM22678TJ-5.0/NOPB
- U6: MPN (none) -> ADP3338AKCZ-3.3-RL
Connections:
- removed net 12V_CLEAN: C10.1, C14.1, C20.POS, C21.POS, C29.1, C30.1, L2.2, R2.1, TP3.P$1, U5.VIN
- new net 12V: 12V.P$1, C10.1, C14.1, C18.POS, C19.POS, C29.1, C30.1, D2.CATHODE, R2.1, U5.VIN
- new net 5V: 5V.P$1, C13.1, C15.POS, C16.1, C17.1, C28.POS, L3.P$1, U5.FB, U6.IN
- new net DOME_PWR: J6.PIN3
- net 12V_BATT: now also J6.PIN1; no longer BOARD_PWR.PIN1
- net 12V_BATT_ON: no longer C18.POS, C19.POS, D2.CATHODE, L2.1, TP4.P$1
- net 3.3V: now also 3.3V.P$1, R11.1; no longer R11.2, TP2.P$1
- net 5V_PWR: no longer C13.1, C15.POS, C16.1, C17.1, C28.POS, L3.P$1, TP1.P$1, U5.FB, U6.IN
- net CHASSIS_GND: no longer BOARD_PWR.PIN2, C18.NEG, C19.NEG, L2.4, TP6.P$1, TVS1.P$1
- net GND: now also C18.NEG, C19.NEG, GND.P$1, J6.PIN2, TVS1.P$1; no longer C20.NEG, C21.NEG, L2.3, TP5.P$1
- net N$9: now also R11.2; no longer R11.1
Other:
- note added: "5V POWER SUPPLY"
- note added: "POWER INPUT"
- moved on the sheet: 3.3V_PWR, C10, C13, C14, C15, C16, C17, C18, C19, C22, C23, C24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
