File: Hardware/Mainboard/Cyclone-Pulse-Wrangler-Mainboard.sch (EAGLE design)
At the start: 61 parts, among them J1 TYPE-C-31-M-12, J2 MF-CON-2.54mm-01x02, J3 MF-CON-2.54mm-01x01, J4 RJHSE-538X, SW1 MF-SW-TACT-4.2MM, U1 ATSAMD21G18A, U2 IP4234CZ6,125, U3 LT8672EMS#PBF, U4 NCP1117DT33G, U5 ACS72981LLRATR-100U3, U6 IPD100N06S403ATMA2, U7 PCA9615DP, X1 ABS25-32.768KHZ-T

Commit message: Initial schematic completed
Parts:
- added C22, C24, C25, C26, C28, C29, C30: 0.1uF, PP_Passives:CAPACITOR_NON_POLAR_0805
- added C23, C27, C31: 1uF, PP_Passives:CAPACITOR_NON_POLAR_0805
- added D6: BZT52C13LPQ-7, PP_Passives:DIODE_SOD-123
- added D7, D8: BZT52C3V6-TP, PP_Passives:DIODE_SOD-123
- added J5, J6: MF-CON-2.54mm-01x06, MF_Connectors:CON_01X06_PTH_2.54MM
- added R10, R11, R12, R9: 0, MF_Passives:RESISTOR_0603
- added R13, R14, R15, R16, R24, R27, R28, R32, R8: 100, MF_Passives:RESISTOR_0603
- added R17, R25: 2.49K, MF_Passives:RESISTOR_0805
- added R18, R26, R33: 2.2K, MF_Passives:RESISTOR_0805
- added R19, R29, R34: 10K, MF_Passives:RESISTOR_0805
- added R20, R22, R23, R30: 10K, MF_Passives:RESISTOR_0603
- added R21, R31: 3.7K, MF_Passives:RESISTOR_0603
- added R35: 3.7K, MF_Passives:RESISTOR_0805
- added U10: SP721ABG, PP_Passives:SP721ABG
- added U8, U9: A2N7002H-HF, PP_DiscreteSemi:MOSFET_N-CHANNEL_SINGLE_SOT-23
- J4: value RJHSE-538X -> RJHSE-538B
Connections:
- removed net A1: U1.PB8/EIC/AIN2/SCOM4PAD0/TC4
- removed net A2: U1.PB9/EIC/AIN3/SCOM4PAD1/TC4
- removed net A3: U1.PA4/EIC/REF/AIN4/SCOM0PAD0/TC0
- removed net D0: U1.PA11/EIC/AIN19/SCOM2PAD3/TC1
- removed net D1: U1.PA10/EIC/AIN18/SCOM2PAD2/TC1
- removed net D2: U1.PA14/XIN/EIC/SCOM2PAD2/TC3
- removed net D3: U1.PA9/I2C/EIC/AIN17/SCOM2PAD1/TC0
- removed net D4: U1.PA8/I2C/AIN16/SCOM2PAD0/TC0
- removed net D5: U1.PA15/XOUT/EIC/SCOM2PAD3/TC3
- new net !A/C_OVERRIDE: C25.2, D7.CATHODE, D8.CATHODE, R20.P$2, R21.P$1, R24.P$1, R24.P$2, R30.P$2, R31.P$1, R32.P$2, U1.PA9/I2C/EIC/AIN17/SCOM2PAD1/TC0, U10.IN_2
- new net !A/C_OVERRIDE_IN: C24.1, J6.PIN3, R19.P$1, R20.P$1
- new net !AUX_DIGITAL: C29.2, R32.P$1, U1.PA15/XOUT/EIC/SCOM2PAD3/TC3, U10.IN_4
- new net !AUX_DIGITAL_IN: C28.1, J6.PIN4, R29.P$1, R30.P$1
- new net AUX_ANALOG: C27.1, R26.P$2, U1.PB9/EIC/AIN3/SCOM4PAD1/TC4, U10.IN_3
- new net AUX_ANALOG_IN: C26.1, C30.1, J5.PIN3, R25.P$1, R26.P$1, R33.P$1, R34.P$1, R35.P$2
- new net BATT_REF: C31.1, R33.P$2, U1.PA4/EIC/REF/AIN4/SCOM0PAD0/TC0
- new net CLT: C23.1, R18.P$2, U1.PB8/EIC/AIN2/SCOM4PAD0/TC4, U10.IN_1
- new net CLT_IN: C22.1, J5.PIN5, R17.P$1, R18.P$1
- new net DM_CONNECTOR: R12.P$2, U2.I/O1A
- new net DM_SCREEN: J4.7, R11.P$2
- new net DP_CONNECTOR: R10.P$2, U2.I/O2A
- new net DP_SCREEN: J4.8, R9.P$2
- new net LED_0: J4.C1, U1.PA14/XIN/EIC/SCOM2PAD2/TC3
- new net LED_1: J4.C0, U1.PA8/I2C/AIN16/SCOM2PAD0/TC0
- new net N$11: J4.A1, R28.P$2
- new net N$12: J4.A0, R27.P$2
- new net N$13: U10.IN_6
- new net N$16: U10.IN_5
- new net N$19: J6.PIN5
- new net N$20: J6.PIN6
- new net N$5: R8.P$1, U3.EN/UVLO
- new net N$6: R13.P$2, R22.P$1, U8.GATE
- new net N$7: R15.P$2, R23.P$1, U9.GATE
- new net P$1: R27.P$1, R28.P$1
- new net PWM_FAN_HI: R15.P$1, U1.PA10/EIC/AIN18/SCOM2PAD2/TC1
- new net PWM_FAN_HI_OUT: J6.PIN2, R16.P$1, U9.DRAIN
- new net PWM_FAN_LO: R13.P$1, U1.PA11/EIC/AIN19/SCOM2PAD3/TC1
- new net PWM_FAN_LO_OUT: J6.PIN1, R14.P$1, U8.DRAIN
- net 12V: now also C24.2, C28.2, D6.CATHODE, R14.P$2, R16.P$2, R19.P$2, R29.P$2
- net 12V_PWR: now also R34.P$2
- net 12V_SW: now also J5.PIN1
- net 3.3V: now also R17.P$2, R25.P$2, U10.V+
- net DM: now also R11.P$1, R12.P$1; no longer U2.I/O1A
- net DP: now also R10.P$1, R9.P$1; no longer U2.I/O2A
- net GND: now also C22.2, C23.2, C25.1, C26.2, C27.2, C29.1, C30.2, C31.2, D6.ANODE, D7.ANODE, D8.ANODE, J5.PIN2, J5.PIN4, J5.PIN6, R21.P$2, R22.P$2, R23.P$2, R31.P$2, R35.P$1, U10.V-, U8.SOURCE, U9.SOURCE
- net N$4: now also R8.P$2; no longer U3.EN/UVLO
Other:
- moved on the sheet: C1, C10, C11, C12, C13, C14, C15, C16, C17, C18, C19, C2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
