File: Hardware/Display-Board/Cyclone-Pulse-Wrangler-Display-Board.sch (EAGLE design)
At the start: 113 parts, among them J1 TYPE-C-31-M-12, J2 MF-CON-2.54mm-01x02, J3 MF-CON-2.54mm-01x01, J4 RJHSE-538B, J5 MF-CON-2.54mm-01x06, J6 MF-CON-2.54mm-01x06, SW1 MF-SW-TACT-4.2MM, U1 ATSAMD21G18A, U10 SP721ABG, U2 IP4234CZ6,125, U3 LT8672EMS#PBF, U4 NCP1117DT33G, U5 ACS72981LLRATR-100U3, U6 IPD100N06S403ATMA2, U7 PCA9615DP, U8 A2N7002H-HF, U9 A2N7002H-HF, X1 ABS25-32.768KHZ-T

Commit message: adding Display board and fixing problems with i2c diff pair
Parts:
- removed C1, C23, C27, C31, C6, C9: 1uF, PP_Passives:CAPACITOR_NON_POLAR_0805
- removed C10: 4.7uF, PP_Passives:CAPACITOR_NON_POLAR_1210
- removed C11, C12, C14, C16, C17, C22, C24, C25, C26, C28, C29, C30, C7: 0.1uF, PP_Passives:CAPACITOR_NON_POLAR_0805
- removed C13: 470uF, PP_Passives:CAPACITOR_POLARIZED_10MM_SMD
- removed C15, C8: 10uF, PP_Passives:CAPACITOR_NON_POLAR_1210
- removed C2, C3: 12pF, PP_Passives:CAPACITOR_NON_POLAR_0805
- removed D1, D2: TPSMB33A, PP_Passives:DIODE_DO-214AA
- removed D3, D4: TPSMB18A, PP_Passives:DIODE_DO-214AA
- removed D6: BZT52C13LPQ-7, PP_Passives:DIODE_SOD-123
- removed D7, D8: BZT52C3V6-TP, PP_Passives:DIODE_SOD-123
- removed F1, F2: (no value), PP_Passives:PTC_FUSE_2920
- removed J5, J6: MF-CON-2.54mm-01x06, MF_Connectors:CON_01X06_PTH_2.54MM
- removed JMP1, R10, R11, R12, R9: 0, MF_Passives:RESISTOR_0603
- removed L1: XPL2010-104MLC, PP_Passives:INDUCTOR_XPL2010
- removed LUG1, LUG2: B4A-PCB-RLM-KIT, PP_Connectors:CON_01X01_B4A-PCB-RLM
- removed R1, R20, R22, R23, R30, R5: 10K, MF_Passives:RESISTOR_0603
- removed R13, R14, R15, R16, R24, R3, R32, R8: 100, MF_Passives:RESISTOR_0603
- removed R17, R25: 2.49K, MF_Passives:RESISTOR_0805
- removed R18, R26, R33: 2.2K, MF_Passives:RESISTOR_0805
- removed R19, R29, R34: 10K, MF_Passives:RESISTOR_0805
- removed R21, R31: 3.7K, MF_Passives:RESISTOR_0603
- removed R35: 3.7K, MF_Passives:RESISTOR_0805
- removed SW1: MF-SW-TACT-4.2MM, MF_Switches:TACT_4.2MM
- removed TC1: TC2030-IDC-NL, MF_Connectors:CON_02X03_SWD2TC_TC2030-IDC-NL
- removed U1: ATSAMD21G18A, PP_DigitalIC:ATSAMD21G18A-AU
- removed U10: SP721ABG, PP_Passives:SP721ABG
- removed U3: LT8672EMS#PBF, PP_PowerIC:LT8672EMS#PBF
- removed U4: NCP1117DT33G, PP_PowerIC:LINEAR_VOTLAGE_REGULATORS_NCP1117DT
- removed U5: ACS72981LLRATR-100U3, PP_Sensors:ACS72981
- removed U6: IPD100N06S403ATMA2, PP_DiscreteSemi:MOSFET_N-CHANNEL_SINGLE_TO-252-3
- removed U8, U9: A2N7002H-HF, PP_DiscreteSemi:MOSFET_N-CHANNEL_SINGLE_SOT-23
- removed X1: ABS25-32.768KHZ-T, MF_Frequency_Control:CYRSTAL_ABS25
- J2: value MF-CON-2.54mm-01x02 -> MF-CON-2.54mm-01x04; device MF_Connectors:CON_01X02_PTH_2.54MM -> MF_Connectors:CON_01X04_PTH_2.54MM
Connections:
- removed net !A/C_OVERRIDE: C25.2, D7.CATHODE, D8.CATHODE, R20.P$2, R21.P$1, R24.P$1, R24.P$2, R30.P$2, R31.P$1, R32.P$2, U1.PA9/I2C/EIC/AIN17/SCOM2PAD1/TC0, U10.IN_2
- removed net !A/C_OVERRIDE_IN: C24.1, J6.PIN3, R19.P$1, R20.P$1
- removed net !AUX_DIGITAL: C29.2, R32.P$1, U1.PA15/XOUT/EIC/SCOM2PAD3/TC3, U10.IN_4
- removed net !AUX_DIGITAL_IN: C28.1, J6.PIN4, R29.P$1, R30.P$1
- removed net !RESET: R1.P$2, R3.P$1, SW1.P$1, TC1.PIN6
- removed net 12V: C10.1, C13.POS, C24.2, C28.2, C9.1, D6.CATHODE, J2.PIN2, JMP1.P$1, L1.P$1, R14.P$2, R16.P$2, R19.P$2, R29.P$2, U3.DRAIN, U6.DRAIN
- removed net 12V_FAN+: LUG2.PIN1, U5.IP-
- removed net 12V_PWR: D1.CATHODE, F1.P$1, LUG1.PIN1, R34.P$2, U5.IP+
- removed net 12V_SW: D2.CATHODE, F2.P$1, J5.PIN1
- removed net A4: U1.PA5/EIC/AIN5/SCOM0PAD1/TC0
- removed net A5: U1.PB2/EIC/AIN10/SCOM5PAD0
- removed net AREF: C6.1, U1.PA3/EIC/REF/AIN1
- removed net AUX_ANALOG: C27.1, R26.P$2, U1.PB9/EIC/AIN3/SCOM4PAD1/TC4, U10.IN_3
- removed net AUX_ANALOG_IN: C26.1, C30.1, J5.PIN3, R25.P$1, R26.P$1, R33.P$1, R34.P$1, R35.P$2
- removed net BATT_REF: C31.1, R33.P$2, U1.PA4/EIC/REF/AIN4/SCOM0PAD0/TC0
- removed net CLT: C23.1, R18.P$2, U1.PB8/EIC/AIN2/SCOM4PAD0/TC4, U10.IN_1
- removed net CLT_IN: C22.1, J5.PIN5, R17.P$1, R18.P$1
- removed net D10: U1.PA18/EIC/SCOM1PAD2/TC3
- removed net D11: U1.PA16/I2C/EIC/SCOM1PAD0/TC1
- removed net D12: U1.PA19/EIC/SCOM1PAD3/TC3
- removed net D13: U1.PA17/I2C/EIC/SCOM1PAD1/TC2
- removed net D18: U1.PA22/I2C/EIC/SCOM5PAD0/TC4
- removed net D19: U1.PA23/I2C/EIC/SCOM5PAD1/TC4
- removed net D6: U1.PA20/EIC/SCOM5PAD2
- removed net D7: U1.PA21/EIC/SCOM5PAD3
- removed net D8: U1.PA6/EIC/AIN6/SCOM0PAD2/TC1
- removed net D9: U1.PA7/EIC/AIN7/SCOM0PAD3/TC1
- removed net DM_CONNECTOR: R12.P$2, U2.I/O1A
- removed net DM_SCREEN: J4.3, R11.P$2
- removed net DP_CONNECTOR: R10.P$2, U2.I/O2A
- removed net DP_SCREEN: J4.6, R9.P$2
- removed net FAN_CURRENT: C17.1, U1.PA2/EIC/AIN0, U5.VIOUT
- removed net N$1: D2.ANODE, D4.ANODE
- removed net N$13: U10.IN_6
- removed net N$14: C9.2, U3.AUX
- removed net N$15: L1.P$2, U3.AUXSW
- removed net N$16: U10.IN_5
- removed net N$19: J6.PIN5
- removed net N$2: U3.GATE, U6.GATE
- removed net N$20: J6.PIN6
- removed net N$3: F1.P$2, U3.SOURCE, U6.SOURCE
- removed net N$4: F2.P$2, R5.P$2, R8.P$2
- removed net N$5: R8.P$1, U3.EN/UVLO
- removed net N$6: R13.P$2, R22.P$1, U8.GATE
- removed net N$7: R15.P$2, R23.P$1, U9.GATE
- removed net N$9: D1.ANODE, D3.ANODE
- removed net PA12: U1.PA12/I2C/EIC/SCOM2PAD0/TC2
- removed net PA13: U1.PA13/I2C/EIC/SCOM2PAD1/TC2
- removed net PA27: U1.PA27/EIC
- removed net PA28: U1.PA28/EIC
- removed net PB22: U1.PB22/EIC/SCOM5PAD2
- removed net PB23: U1.PB23/EIC/SCOM5PAD3
- removed net PB3: U1.PB3/EIC/AIN11/SCOM5PAD1
- removed net PWM_FAN_HI: R15.P$1, U1.PA10/EIC/AIN18/SCOM2PAD2/TC1
- removed net PWM_FAN_HI_OUT: J6.PIN2, R16.P$1, U9.DRAIN
- removed net PWM_FAN_LO: R13.P$1, U1.PA11/EIC/AIN19/SCOM2PAD3/TC1
- removed net PWM_FAN_LO_OUT: J6.PIN1, R14.P$1, U8.DRAIN
- removed net REG_INPUT: C8.1, J2.PIN1, JMP1.P$2, U4.IN
- removed net RESETLIN: R3.P$2, U1.!RESET
- removed net SCL_SCREEN: R6.P$1, U1.PB11/EIC/SCOM4PAD3/TC5, U7.SCL
- removed net SDA_SCREEN: R7.P$1, U1.PB10/EIC/SCOM4PAD2/TC5, U7.SDA
- removed net SWCLK: TC1.PIN4, U1.PA30/EIC/SCOM1PAD2/TC1
- removed net SWDIO: TC1.PIN3, U1.PA31/EIC/SCOM1PAD3/TC1
- removed net SWO: TC1.PIN5
- removed net VDDCORE: C1.1, U1.VDDCORE1
- removed net XIN32: C2.2, U1.PA0/XIN32/EIC/SCOM1PAD0/TC2, X1.X0
- removed net XOUT32: C3.2, U1.PA1/XOUT32/EIC/SCOM1PAD1/TC2, X1.X1
- new net SCL: J2.PIN2, R6.P$1, U7.SCL
- new net SDA: J2.PIN1, R7.P$1, U7.SDA
- net 3.3V: now also J2.PIN3; no longer C11.1, C12.1, C14.1, C15.1, C16.1, C7.1, R1.P$1, R17.P$2, R25.P$2, TC1.PIN1, U1.VDDANA, U1.VDDIN, U1.VDDIO1, U1.VDDIO2, U10.V+, U4.OUT, U5.VCC
- net DM: now also J4.3, U2.I/O1A; no longer R11.P$1, R12.P$1, U1.PA24/EIC/SCOM3PAD2/TC5
- net DP: now also J4.6, U2.I/O2A; no longer R10.P$1, R9.P$1, U1.PA25/EIC/SCOM3PAD3/TC5
- net GND: now also J2.PIN4; no longer C1.2, C10.2, C11.2, C12.2, C13.NEG, C14.2, C15.2, C16.2, C17.2, C2.1, C22.2, C23.2, C25.1, C26.2, C27.2, C29.1, C3.1, C30.2, C31.2, C6.2, C7.2, C8.2, D3.CATHODE, D4.CATHODE, D6.ANODE, D7.ANODE, D8.ANODE, J5.PIN2, J5.PIN4, J5.PIN6, R21.P$2, R22.P$2, R23.P$2, R31.P$2, R35.P$1, R5.P$1, SW1.P$3, TC1.PIN2, U1.GND, U10.V-, U3.GND, U4.GND, U5.GND, U8.SOURCE, U9.SOURCE
- net LED_0: no longer U1.PA14/XIN/EIC/SCOM2PAD2/TC3
- net LED_1: no longer U1.PA8/I2C/AIN16/SCOM2PAD0/TC0
Other:
- moved on the sheet: C18, C19, C20, C21, C4, C5, D5, F3, J1, J3, J4, L2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
